File: hardware/pcb/kicad/coluna_2u.kicad_pcb (KiCad board)
At the start: 2 copper layers, 35.4 x 89.5 mm, 30 parts

Commit message: Placas rev0 roteadas: route.py (Freerouting + DRC), LEDs na placa L, diodos SOD-123
- route.py termina as placas do Ergogen no KiCad 10: regras da JLCPCB,
  diodo SOD-123 na face de baixo, 3 LEDs 0805 + resistores na placa L,
  área proibida no furo da trava, roteamento pelo Freerouting e DRC.
- As três placas saem com DRC limpo (0 violações, 0 ligações faltando).
- Barra do polegar com switches girados 180°: o pino 2 ficava a 0,28 mm
  da borda de trás.
- Prévia com trilhas, vias e LEDs; lê o formato atual do KiCad.
- CAD: LEDs com tamanho 0805. Sem colisões (gav_fixed, lboard_parts,
  lboard_gav em 0 e 150%).

Co-Authored-By: Claude Opus 5.5 <noreply@anthropic.com>
Parts:
- D1, D10, D2, D3, D4, D5, D6, D7, D8, D9: value (none) -> 1N4148W; footprint ComboDiode -> D_SOD-123; moved to B.Cu
Routing:
- net C2: track 0.00 -> 103.9 mm
- net C1: track 0.00 -> 91.2 mm
- net R4: track 0.00 -> 90.9 mm, vias 0 -> 2
- net R3: track 0.00 -> 71.9 mm, vias 0 -> 2
- net R2: track 0.00 -> 55.1 mm, vias 0 -> 2
- net R1: track 0.00 -> 39.1 mm, vias 0 -> 2
- net R0: track 0.00 -> 27.1 mm
- net c1_r2: track 0.00 -> 13.7 mm, vias 0 -> 1
- net c1_r3: track 0.00 -> 13.3 mm, vias 0 -> 1
- net c1_r1: track 0.00 -> 13.2 mm, vias 0 -> 1
- net c1_r4: track 0.00 -> 12.5 mm
- net c1_r0: track 0.00 -> 12.5 mm, vias 0 -> 1
- net c2_r0: track 0.00 -> 12.4 mm
- net c2_r4: track 0.00 -> 12.4 mm
- net c2_r1: track 0.00 -> 12.4 mm
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Other:
- net class Default removed

Commit message: Metade esquerda num arquivo só (assemble.py) e placas centralizadas na folha
- assemble.py junta placa L + 3 colunas 1u + coluna 2u na posição do CAD
  (ortho e stagger 150%), com as redes reais da matriz; os jumpers viram
  linhas de ligação. As 34 ligações pendentes batem com o barramento.
- route.py centraliza cada placa na folha A3; a prévia alinha pelo contorno.

Co-Authored-By: Claude Opus 5.5 <noreply@anthropic.com>
Parts:
- moved D1 273.0 mm to (201.0, 190.1)
- moved D10 273.0 mm to (219.0, 117.5)
- moved D2 273.0 mm to (201.0, 173.1)
- moved D3 273.0 mm to (201.0, 156.1)
- moved D4 273.0 mm to (201.0, 139.1)
- moved D5 273.0 mm to (201.0, 117.5)
- moved D6 273.0 mm to (219.0, 190.1)
- moved D7 273.0 mm to (219.0, 173.1)
- moved D8 273.0 mm to (219.0, 156.1)
- moved D9 273.0 mm to (219.0, 139.1)
- moved PAD1 273.0 mm to (194.0, 122.4)
- moved PAD10 273.0 mm to (199.1, 123.6)
- moved PAD2 273.0 mm to (195.3, 122.4)
- moved PAD3 273.0 mm to (196.5, 122.4)
- moved PAD4 273.0 mm to (197.8, 122.4)
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