File: hardware/pcb/kicad/coluna_1u.kicad_pcb (KiCad board)
At the start: 2 copper layers, 17.4 x 89.5 mm, 29 parts

Commit message: Placas rev0 roteadas: route.py (Freerouting + DRC), LEDs na placa L, diodos SOD-123
- route.py termina as placas do Ergogen no KiCad 10: regras da JLCPCB,
  diodo SOD-123 na face de baixo, 3 LEDs 0805 + resistores na placa L,
  área proibida no furo da trava, roteamento pelo Freerouting e DRC.
- As três placas saem com DRC limpo (0 violações, 0 ligações faltando).
- Barra do polegar com switches girados 180°: o pino 2 ficava a 0,28 mm
  da borda de trás.
- Prévia com trilhas, vias e LEDs; lê o formato atual do KiCad.
- CAD: LEDs com tamanho 0805. Sem colisões (gav_fixed, lboard_parts,
  lboard_gav em 0 e 150%).

Co-Authored-By: Claude Opus 5.5 <noreply@anthropic.com>
Parts:
- D1, D2, D3, D4, D5: value (none) -> 1N4148W; footprint ComboDiode -> D_SOD-123; moved to B.Cu
Routing:
- net C1: track 0.00 -> 95.0 mm
- net R4: track 0.00 -> 86.7 mm, vias 0 -> 2
- net R3: track 0.00 -> 64.9 mm, vias 0 -> 3
- net R2: track 0.00 -> 49.3 mm, vias 0 -> 3
- net R1: track 0.00 -> 44.6 mm, vias 0 -> 4
- net c1_r1: track 0.00 -> 17.5 mm
- net R0: track 0.00 -> 14.4 mm
- net C3: track 0.00 -> 12.7 mm, vias 0 -> 4
- net c1_r2: track 0.00 -> 12.5 mm
- net c1_r4: track 0.00 -> 12.5 mm
- net c1_r0: track 0.00 -> 12.5 mm
- net c1_r3: track 0.00 -> 12.4 mm
- net C4: track 0.00 -> 10.2 mm, vias 0 -> 2
- net C2: track 0.00 -> 10.0 mm
- net C5: track 0.00 -> 9.65 mm, vias 0 -> 2
Other:
- net class Default removed

Commit message: Metade esquerda num arquivo só (assemble.py) e placas centralizadas na folha
- assemble.py junta placa L + 3 colunas 1u + coluna 2u na posição do CAD
  (ortho e stagger 150%), com as redes reais da matriz; os jumpers viram
  linhas de ligação. As 34 ligações pendentes batem com o barramento.
- route.py centraliza cada placa na folha A3; a prévia alinha pelo contorno.

Co-Authored-By: Claude Opus 5.5 <noreply@anthropic.com>
Parts:
- moved D1 279.7 mm to (210.0, 190.1)
- moved D2 279.7 mm to (210.0, 173.1)
- moved D3 279.7 mm to (210.0, 156.1)
- moved D4 279.7 mm to (210.0, 139.1)
- moved D5 279.7 mm to (210.0, 117.5)
- moved PAD1 279.7 mm to (203.0, 122.4)
- moved PAD10 279.7 mm to (208.1, 123.6)
- moved PAD11 279.7 mm to (211.9, 122.4)
- moved PAD12 279.7 mm to (213.2, 122.4)
- moved PAD13 279.7 mm to (214.4, 122.4)
- moved PAD14 279.7 mm to (215.7, 122.4)
- moved PAD15 279.7 mm to (217.0, 122.4)
- moved PAD16 279.7 mm to (211.9, 123.6)
- moved PAD17 279.7 mm to (213.2, 123.6)
- moved PAD18 279.7 mm to (214.4, 123.6)
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
Commit message: LED RGB por tecla, mão direita e teclado inteiro num arquivo
- LED RGB SK6812MINI-E em cada tecla Choc (38 + 35), na janela do Choc;
  diodos vão para o canto noroeste; capacitor de 4,7 uF por placa.
- Jumper de 13 vias (linhas, colunas, VLED, GND, DAT) em blocos 2 x 7,
  J_IN e J_OUT em alturas diferentes; cabeçalho da placa L com 20 pads.
- Mão direita: placa_L_dir (8 teclas 1u + shift 2u; barra com espaço,
  return, cmd e 4 setas táteis TS-1187A), coluna_1u_dir, coluna_2u_dir.
- As 6 placas roteadas com DRC limpo; regra de borda de 0,5 mm com
  exceção de 0,2 mm só para os pads do LED junto do próprio recorte.
- assemble.py monta o teclado inteiro (teclado_150 e teclado_0); as 92
  ligações pendentes são exatamente os jumpers.
- CAD: blocos de pads e jumpers novos, sem colisões em 0 e 150%.

Co-Authored-By: Claude Opus 5.5 <noreply@anthropic.com>
Parts:
- added C1: 4.7uF, C_0805_2012Metric, B.Cu at (216.3, 176.2)
- added L1: SK6812MINI-E, LED_SK6812MINI-E_3.2x2.8mm_P1.5mm_ReverseMount, B.Cu at (210.0, 117.0)
- added L2: SK6812MINI-E, LED_SK6812MINI-E_3.2x2.8mm_P1.5mm_ReverseMount, B.Cu at (210.0, 138.4)
- added L3: SK6812MINI-E, LED_SK6812MINI-E_3.2x2.8mm_P1.5mm_ReverseMount, B.Cu at (210.0, 155.4)
- added L4: SK6812MINI-E, LED_SK6812MINI-E_3.2x2.8mm_P1.5mm_ReverseMount, B.Cu at (210.0, 172.4)
- added L5: SK6812MINI-E, LED_SK6812MINI-E_3.2x2.8mm_P1.5mm_ReverseMount, B.Cu at (210.0, 189.4)
- added PAD20: , SMDPad, F.Cu at (217.4, 124.0)
- added PAD21: , SMDPad, F.Cu at (209.8, 125.2)
- added PAD22: , SMDPad, F.Cu at (211.1, 125.2)
- added PAD23: , SMDPad, F.Cu at (212.3, 125.2)
- added PAD24: , SMDPad, F.Cu at (213.6, 125.2)
- added PAD25: , SMDPad, F.Cu at (216.1, 125.2)
- moved D1 10.4 mm to (206.4, 180.2), turned to 90 degrees
- moved D2 10.4 mm to (206.4, 163.2), turned to 90 degrees
- moved D3 10.4 mm to (206.4, 146.2), turned to 90 degrees
- moved D4 10.4 mm to (206.4, 129.2), turned to 90 degrees
- moved D5 10.4 mm to (206.4, 107.8), turned to 90 degrees
- moved PAD6 6.61 mm to (208.9, 120.8)
- moved PAD7 6.61 mm to (210.2, 120.8)
- moved PAD14 6.14 mm to (209.8, 124.0)
- moved PAD15 6.14 mm to (211.1, 124.0)
- moved PAD11 5.50 mm to (206.4, 122.0)
- moved PAD13 5.50 mm to (208.9, 122.0)
- moved PAD12 5.50 mm to (207.7, 122.0)
- moved PAD10 3.35 mm to (205.1, 122.0)
- moved PAD8 3.35 mm to (202.6, 122.0)
- moved PAD9 3.35 mm to (203.9, 122.0)
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Connections:
- PAD10 pad 1: C5 -> C3
- PAD11 pad 1: R0 -> C4
- PAD12 pad 1: R1 -> C5
- PAD13 pad 1: R2 -> DIN
- PAD14 pad 1: R3 -> R0
- PAD15 pad 1: R4 -> R1
- PAD16 pad 1: C2 -> R2
- PAD17 pad 1: C3 -> R3
- PAD18 pad 1: C4 -> R4
- PAD19 pad 1: C5 -> VLED
- PAD6 pad 1: C1 -> VLED
- PAD7 pad 1: C2 -> GND
- PAD8 pad 1: C3 -> C1
- PAD9 pad 1: C4 -> C2
Routing:
- net GND: track 0.00 -> 121.1 mm, vias 0 -> 7
- net VLED: track 0.00 -> 94.2 mm, vias 0 -> 6
- net DOUT: track 0.00 -> 66.3 mm
- net rgb1: track 0.00 -> 34.2 mm, vias 0 -> 2
- net DIN: track 0.00 -> 31.1 mm, vias 0 -> 2
- net rgb4: track 0.00 -> 27.2 mm, vias 0 -> 2
- net rgb3: track 0.00 -> 23.1 mm, vias 0 -> 2
- net rgb2: track 0.00 -> 22.6 mm
- net R1: track 44.6 -> 25.8 mm
- net c1_r1: track 17.5 -> 3.70 mm
- net R0: track 14.4 -> 26.4 mm, vias 0 -> 2
- net R4: track 86.7 -> 75.0 mm, vias 2 -> 0
- net R2: track 49.3 -> 39.7 mm
- net c1_r2: track 12.5 -> 3.70 mm
- net c1_r4: track 12.5 -> 3.70 mm
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