File: hardware/pcb/kicad/coluna_2u_dir.kicad_pcb (KiCad board)
At the start: 2 copper layers, 35.4 x 89.5 mm, 44 parts

Commit message: LED RGB por tecla, mão direita e teclado inteiro num arquivo
- LED RGB SK6812MINI-E em cada tecla Choc (38 + 35), na janela do Choc;
  diodos vão para o canto noroeste; capacitor de 4,7 uF por placa.
- Jumper de 13 vias (linhas, colunas, VLED, GND, DAT) em blocos 2 x 7,
  J_IN e J_OUT em alturas diferentes; cabeçalho da placa L com 20 pads.
- Mão direita: placa_L_dir (8 teclas 1u + shift 2u; barra com espaço,
  return, cmd e 4 setas táteis TS-1187A), coluna_1u_dir, coluna_2u_dir.
- As 6 placas roteadas com DRC limpo; regra de borda de 0,5 mm com
  exceção de 0,2 mm só para os pads do LED junto do próprio recorte.
- assemble.py monta o teclado inteiro (teclado_150 e teclado_0); as 92
  ligações pendentes são exatamente os jumpers.
- CAD: blocos de pads e jumpers novos, sem colisões em 0 e 150%.

Co-Authored-By: Claude Opus 5.5 <noreply@anthropic.com>
Parts:
- moved PAD1 32.8 mm to (226.4, 120.8)
- moved PAD8 32.8 mm to (226.4, 122.0)
- moved PAD2 30.3 mm to (225.1, 120.8)
- moved PAD9 30.3 mm to (225.1, 122.0)
- moved PAD10 27.7 mm to (223.9, 122.0)
- moved PAD3 27.7 mm to (223.9, 120.8)
- moved PAD11 25.2 mm to (222.6, 122.0)
- moved PAD4 25.2 mm to (222.6, 120.8)
- moved PAD12 22.6 mm to (221.3, 122.0)
- moved PAD5 22.6 mm to (221.3, 120.8)
- moved PAD13 20.1 mm to (220.1, 122.0)
- moved PAD6 20.1 mm to (220.1, 120.8)
- moved D1 18.0 mm to (215.4, 180.2)
- moved D10 18.0 mm to (197.4, 107.8)
- moved D2 18.0 mm to (215.4, 163.2)
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Routing:
- net rgb1: track 13.2 -> 34.4 mm
- net VLED: track 179.3 -> 196.1 mm
- net rgb6: track 29.1 -> 13.2 mm
- net R4: track 83.7 -> 98.7 mm
- net rgb5: track 22.5 -> 36.2 mm
- net R2: track 48.3 -> 58.2 mm
- net GND: track 213.0 -> 204.3 mm, vias 10 -> 8
- net R0: track 32.0 -> 39.9 mm, vias 2 -> 0
- net C2: track 105.5 -> 98.5 mm
- net C1: track 92.6 -> 85.6 mm
- net R1: track 31.7 -> 35.9 mm
- net R3: track 65.9 -> 68.3 mm
- net rgb4: track 23.4 -> 25.6 mm, vias 2 -> 0
- net rgb7: track 21.0 -> 19.0 mm
- net rgb2: track 28.7 -> 27.1 mm
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