File: hardware/pcb/kicad/placa_L.kicad_pcb (KiCad board)
At the start: 2 copper layers, 124.7 x 105.5 mm, 54 parts

Commit message: Placas rev0 roteadas: route.py (Freerouting + DRC), LEDs na placa L, diodos SOD-123
- route.py termina as placas do Ergogen no KiCad 10: regras da JLCPCB,
  diodo SOD-123 na face de baixo, 3 LEDs 0805 + resistores na placa L,
  área proibida no furo da trava, roteamento pelo Freerouting e DRC.
- As três placas saem com DRC limpo (0 violações, 0 ligações faltando).
- Barra do polegar com switches girados 180°: o pino 2 ficava a 0,28 mm
  da borda de trás.
- Prévia com trilhas, vias e LEDs; lê o formato atual do KiCad.
- CAD: LEDs com tamanho 0805. Sem colisões (gav_fixed, lboard_parts,
  lboard_gav em 0 e 150%).

Co-Authored-By: Claude Opus 5.5 <noreply@anthropic.com>
Parts:
- added LED1: LED 0805, LED_0805_2012Metric, F.Cu at (-5.00, -61.8)
- added LED2: LED 0805, LED_0805_2012Metric, F.Cu at (0.00, -61.8)
- added LED3: LED 0805, LED_0805_2012Metric, F.Cu at (5.00, -61.8)
- added R1: 1k, R_0805_2012Metric, B.Cu at (-5.00, -61.8)
- added R2: 1k, R_0805_2012Metric, B.Cu at (0.00, -61.8)
- added R3: 1k, R_0805_2012Metric, B.Cu at (5.00, -61.8)
- D1, D10, D11, D12, D13, D2, D3, D4, D5, D6, D7, D8, D9: value (none) -> 1N4148W; footprint ComboDiode -> D_SOD-123; moved to B.Cu
- moved D10 10.6 mm to (36.0, 11.7)
- moved D11 10.6 mm to (54.0, 11.7)
- moved D12 10.6 mm to (76.5, 11.7)
- moved D13 10.6 mm to (103.5, 11.7)
- moved D8 10.6 mm to (0.00, 11.7)
- moved D9 10.6 mm to (18.0, 11.7)
- turned S10 to 180 degrees
- turned S11 to 180 degrees
- turned S12 to 180 degrees
- turned S13 to 180 degrees
- turned S8 to 180 degrees
- turned S9 to 180 degrees
Routing:
- net COL5: track 0.00 -> 180.3 mm, vias 0 -> 2
- net COL4: track 0.00 -> 152.6 mm, vias 0 -> 2
- net COL3: track 0.00 -> 147.8 mm, vias 0 -> 3
- net COL0: track 0.00 -> 133.1 mm, vias 0 -> 2
- net COL1: track 0.00 -> 129.4 mm, vias 0 -> 2
- net R5: track 0.00 -> 127.3 mm, vias 0 -> 6
- net COL2: track 0.00 -> 121.7 mm, vias 0 -> 1
- net R0: track 0.00 -> 117.8 mm, vias 0 -> 4
- net R3: track 0.00 -> 97.1 mm, vias 0 -> 3
- net R2: track 0.00 -> 94.8 mm, vias 0 -> 2
- net R1: track 0.00 -> 93.8 mm, vias 0 -> 3
- net R4: track 0.00 -> 93.5 mm, vias 0 -> 2
- net GND: track 0.00 -> 85.6 mm, vias 0 -> 3
- net COL6: track 0.00 -> 71.9 mm, vias 0 -> 2
- net LED3: track 0.00 -> 59.6 mm
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Other:
- net class Default removed

Commit message: Metade esquerda num arquivo só (assemble.py) e placas centralizadas na folha
- assemble.py junta placa L + 3 colunas 1u + coluna 2u na posição do CAD
  (ortho e stagger 150%), com as redes reais da matriz; os jumpers viram
  linhas de ligação. As 34 ligações pendentes batem com o barramento.
- route.py centraliza cada placa na folha A3; a prévia alinha pelo contorno.

Co-Authored-By: Claude Opus 5.5 <noreply@anthropic.com>
Parts:
- moved D1 236.0 mm to (165.3, 182.1)
- moved D10 236.0 mm to (192.3, 188.4)
- moved D11 236.0 mm to (210.3, 188.4)
- moved D12 236.0 mm to (232.8, 188.4)
- moved D13 236.0 mm to (259.9, 188.4)
- moved D2 236.0 mm to (165.3, 165.1)
- moved D3 236.0 mm to (165.3, 148.1)
- moved D4 236.0 mm to (156.3, 131.1)
- moved D5 236.0 mm to (156.3, 109.5)
- moved D6 236.0 mm to (174.3, 131.1)
- moved D7 236.0 mm to (174.3, 109.5)
- moved D8 236.0 mm to (156.3, 188.4)
- moved D9 236.0 mm to (174.3, 188.4)
- moved LED1 236.0 mm to (151.3, 115.0)
- moved LED2 236.0 mm to (156.3, 115.0)
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Routing:
- net R2: track 94.8 -> 95.3 mm
Other:
- outline, holes or cut-outs redrawn

Commit message: LED RGB por tecla, mão direita e teclado inteiro num arquivo
- LED RGB SK6812MINI-E em cada tecla Choc (38 + 35), na janela do Choc;
  diodos vão para o canto noroeste; capacitor de 4,7 uF por placa.
- Jumper de 13 vias (linhas, colunas, VLED, GND, DAT) em blocos 2 x 7,
  J_IN e J_OUT em alturas diferentes; cabeçalho da placa L com 20 pads.
- Mão direita: placa_L_dir (8 teclas 1u + shift 2u; barra com espaço,
  return, cmd e 4 setas táteis TS-1187A), coluna_1u_dir, coluna_2u_dir.
- As 6 placas roteadas com DRC limpo; regra de borda de 0,5 mm com
  exceção de 0,2 mm só para os pads do LED junto do próprio recorte.
- assemble.py monta o teclado inteiro (teclado_150 e teclado_0); as 92
  ligações pendentes são exatamente os jumpers.
- CAD: blocos de pads e jumpers novos, sem colisões em 0 e 150%.

Co-Authored-By: Claude Opus 5.5 <noreply@anthropic.com>
Parts:
- added C1: 4.7uF, C_0805_2012Metric, B.Cu at (151.8, 168.2)
- added L1: SK6812MINI-E, LED_SK6812MINI-E_3.2x2.8mm_P1.5mm_ReverseMount, B.Cu at (156.3, 189.1)
- added L10: SK6812MINI-E, LED_SK6812MINI-E_3.2x2.8mm_P1.5mm_ReverseMount, B.Cu at (156.3, 130.4)
- added L11: SK6812MINI-E, LED_SK6812MINI-E_3.2x2.8mm_P1.5mm_ReverseMount, B.Cu at (174.3, 130.4)
- added L12: SK6812MINI-E, LED_SK6812MINI-E_3.2x2.8mm_P1.5mm_ReverseMount, B.Cu at (174.3, 109.0)
- added L13: SK6812MINI-E, LED_SK6812MINI-E_3.2x2.8mm_P1.5mm_ReverseMount, B.Cu at (156.3, 109.0)
- added L2: SK6812MINI-E, LED_SK6812MINI-E_3.2x2.8mm_P1.5mm_ReverseMount, B.Cu at (165.3, 181.4)
- added L3: SK6812MINI-E, LED_SK6812MINI-E_3.2x2.8mm_P1.5mm_ReverseMount, B.Cu at (174.3, 189.1)
- added L4: SK6812MINI-E, LED_SK6812MINI-E_3.2x2.8mm_P1.5mm_ReverseMount, B.Cu at (192.3, 189.1)
- added L5: SK6812MINI-E, LED_SK6812MINI-E_3.2x2.8mm_P1.5mm_ReverseMount, B.Cu at (210.3, 189.1)
- added L6: SK6812MINI-E, LED_SK6812MINI-E_3.2x2.8mm_P1.5mm_ReverseMount, B.Cu at (232.8, 189.1)
- added L7: SK6812MINI-E, LED_SK6812MINI-E_3.2x2.8mm_P1.5mm_ReverseMount, B.Cu at (259.9, 189.1)
- added L8: SK6812MINI-E, LED_SK6812MINI-E_3.2x2.8mm_P1.5mm_ReverseMount, B.Cu at (165.3, 164.4)
- added L9: SK6812MINI-E, LED_SK6812MINI-E_3.2x2.8mm_P1.5mm_ReverseMount, B.Cu at (165.3, 147.4)
- added PAD29: , SMDPad, F.Cu at (149.6, 163.7)
- added PAD30: , SMDPad, F.Cu at (149.6, 162.4)
- added PAD31: , SMDPad, F.Cu at (149.6, 161.2)
- added PAD32: , SMDPad, F.Cu at (149.6, 159.9)
- added PAD33: , SMDPad, F.Cu at (149.6, 158.6)
- moved PAD11 71.4 mm to (177.9, 117.2)
- moved PAD12 70.8 mm to (179.2, 117.2)
- moved PAD13 70.2 mm to (180.5, 117.2)
- moved D1 10.4 mm to (161.8, 172.2), turned to 90 degrees
- moved D10 10.4 mm to (195.9, 198.2), turned to 90 degrees
- moved D11 10.4 mm to (213.9, 198.2), turned to 90 degrees
- moved D12 10.4 mm to (236.4, 198.2), turned to 90 degrees
- moved D2 10.4 mm to (161.8, 155.2), turned to 90 degrees
- moved D3 10.4 mm to (161.8, 138.2), turned to 90 degrees
- moved D4 10.4 mm to (152.8, 121.2), turned to 90 degrees
- moved D6 10.4 mm to (170.8, 121.2), turned to 90 degrees
- moved D8 10.4 mm to (159.9, 198.2), turned to 90 degrees
- moved D9 10.4 mm to (177.9, 198.2), turned to 90 degrees
- moved D13 10.4 mm to (263.4, 198.2), turned to 90 degrees
- moved D5 10.4 mm to (152.8, 99.8), turned to 90 degrees
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Connections:
- PAD10 pad 1: COL6 -> COL4
- PAD11 pad 1: GND -> COL5
- PAD12 pad 1: R0 -> COL6
- PAD13 pad 1: R1 -> DOUT
- PAD14 pad 1: R2 -> GND
- PAD15 pad 1: R3 -> VLED
- PAD16 pad 1: R4 -> DIN
- PAD17 pad 1: R5 -> R0
- PAD18 pad 1: COL0 -> R1
- PAD19 pad 1: COL1 -> R2
- PAD20 pad 1: COL2 -> R3
- PAD21 pad 1: COL3 -> R4
- PAD22 pad 1: COL4 -> R5
- PAD23 pad 1: COL5 -> COL0
- PAD24 pad 1: COL6 -> COL1
- PAD25 pad 1: LED1 -> COL2
- PAD26 pad 1: LED2 -> COL3
- PAD27 pad 1: LED3 -> COL4
- PAD28 pad 1: GND -> COL5
- PAD6 pad 1: COL2 -> VLED
- PAD7 pad 1: COL3 -> GND
- PAD8 pad 1: COL4 -> COL2
- PAD9 pad 1: COL5 -> COL3
Routing:
- net GND: track 85.6 -> 393.3 mm, vias 3 -> 12
- net VLED: track 0.00 -> 292.5 mm, vias 0 -> 15
- net rgb7: track 0.00 -> 119.3 mm, vias 0 -> 2
- net rgb12: track 0.00 -> 45.9 mm, vias 0 -> 2
- net rgb6: track 0.00 -> 44.7 mm, vias 0 -> 2
- net rgb5: track 0.00 -> 39.3 mm
- net rgb4: track 0.00 -> 37.2 mm, vias 0 -> 4
- net rgb3: track 0.00 -> 34.9 mm
- net rgb9: track 0.00 -> 30.0 mm, vias 0 -> 2
- net DOUT: track 0.00 -> 28.7 mm, vias 0 -> 2
- net rgb11: track 0.00 -> 28.7 mm, vias 0 -> 2
- net R5: track 127.3 -> 152.3 mm
- net rgb1: track 0.00 -> 18.0 mm, vias 0 -> 2
- net rgb8: track 0.00 -> 17.8 mm
- net COL5: track 180.3 -> 197.9 mm, vias 2 -> 3
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